File: lab3/PCB Design Lab/PCB Design Lab.kicad_sch (KiCad schematic)
At the start: 15 parts, among them J1 Conn_01x04_Pin, U1 TPS79301DBVR, U2 LSM6DSOXTR

Commit message: PCB update
Parts:
- C2: value 2.2µF -> 2.2uF
- C3: value 1µF -> 1uF
- C4: value 0.01µF -> 0.01uF
- U1: footprint TPS79301DBVR:SOT95P280X145-6N -> TPS79301:SOT95P280X145-6N
- U2: footprint LSM6DSOXTR:PQFN50P250X300X86-14N -> LSM6DSOX:PQFN50P250X300X86-14N
Changed lines of the file:
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@@
 			)
 		)
-		(property "Value" "1µF"
+		(property "Value" "1uF"
 			(at 64.77 53.3399 0)
 			(effects
@@
 			)
 		)
-		(property "Footprint" "LSM6DSOXTR:PQFN50P250X300X86-14N"
+		(property "Footprint" "LSM6DSOX:PQFN50P250X300X86-14N"
 			(at 97.79 134.62 0)
 			(effects
@@
 			)
 		)
-		(property "Footprint" "TPS79301DBVR:SOT95P280X145-6N"
+		(property "Footprint" "TPS79301:SOT95P280X145-6N"
 			(at 93.98 55.88 0)
 			(effects
@@
 			)
 		)
-		(property "Value" "2.2µF"
+		(property "Value" "2.2uF"
 			(at 140.97 53.3399 0)
 			(effects
@@
 			)
 		)
-		(property "Value" "0.01µF"
+		(property "Value" "0.01uF"
 			(at 73.66 60.9599 0)
 			(effects
